File: eSim-2.1/Examples/InvertingAmplifier/lm_741.sch (KiCad schematic (older format))
At the start: 33 parts, among them Q1 eSim_NPN, Q10 eSim_PNP, Q11 eSim_PNP, Q12 eSim_NPN, Q13 eSim_NPN, Q14 eSim_NPN, Q15 eSim_NPN, Q16 eSim_NPN, Q17 eSim_NPN, Q18 eSim_NPN, Q19 eSim_PNP, Q2 eSim_NPN, Q20 eSim_NPN, Q3 eSim_NPN, Q4 eSim_PNP, Q5 eSim_PNP, Q6 eSim_PNP, Q7 eSim_NPN, Q8 eSim_NPN, Q9 eSim_PNP, U1 PORT

Commit message: Revert "Added gaw"
This reverts commit 7f7a056778eff9853150f303c9f86ac897313991.
Parts:
- Q1, Q12, Q13, Q14, Q15, Q16, Q17, Q18, Q2, Q20, Q3, Q7, Q8: symbol eSim_NPN -> eSim_NPN-RESCUE-lm_741
- Q10, Q11, Q19, Q4, Q5, Q6, Q9: symbol eSim_PNP -> eSim_PNP-RESCUE-lm_741
Changed lines of the file:
@@
 EESchema Schematic File Version 2
+LIBS:lm_741-rescue
 LIBS:power
 LIBS:eSim_Analog
@@
 LIBS:eSim_Plot
 LIBS:eSim_Power
-LIBS:eSim_PSpice
+LIBS:eSim_User
 LIBS:eSim_Sources
 LIBS:eSim_Subckt
-LIBS:eSim_User
 LIBS:lm_741-cache
 EELAYER 25 0
@@
 $EndDescr
 $Comp
-L eSim_NPN Q1
+L eSim_NPN-RESCUE-lm_741 Q1
 U 1 1 5CE90A7B
 P 2650 2700
@@
 $EndComp
 $Comp
-L eSim_NPN Q2
+L eSim_NPN-RESCUE-lm_741 Q2
 U 1 1 5CE90A7C
 P 4300 2700
@@
 $EndComp
 $Comp
-L eSim_PNP Q6
+L eSim_PNP-RESCUE-lm_741 Q6
 U 1 1 5CE90A7D
 P 3000 3200
@@
 $EndComp
 $Comp
-L eSim_PNP Q5
+L eSim_PNP-RESCUE-lm_741 Q5
 U 1 1 5CE90A7E
 P 3950 3200
@@
 $EndComp
 $Comp
-L eSim_NPN Q3
+L eSim_NPN-RESCUE-lm_741 Q3
 U 1 1 5CE90A7F
 P 3300 4000
@@
 $EndComp
 $Comp
-L eSim_PNP Q4
+L eSim_PNP-RESCUE-lm_741 Q4
 U 1 1 5CE90A80
 P 3850 2000
@@
 $EndComp
 $Comp
-L eSim_PNP Q9
+L eSim_PNP-RESCUE-lm_741 Q9
 U 1 1 5CE90A81
 P 5200 2000
@@
 $EndComp
 $Comp
-L eSim_NPN Q8
+L eSim_NPN-RESCUE-lm_741 Q8
 U 1 1 5CE90A82
 P 3950 4600
@@
 $EndComp
 $Comp
-L eSim_NPN Q7
+L eSim_NPN-RESCUE-lm_741 Q7
 U 1 1 5CE90A83
 P 3000 4600
@@
 $EndComp
 $Comp
-L eSim_NPN Q12
+L eSim_NPN-RESCUE-lm_741 Q12
 U 1 1 5CE90A87
 P 6300 4700
@@
 $EndComp
 $Comp
-L eSim_NPN Q13
+L eSim_NPN-RESCUE-lm_741 Q13
 U 1 1 5CE90A88
 P 5400 4700
@@
 $EndComp
 $Comp
-L eSim_PNP Q10
+L eSim_PNP-RESCUE-lm_741 Q10
 U 1 1 5CE90A8B
 P 6500 1950
@@
 $EndComp
 $Comp
-L eSim_PNP Q11
+L eSim_PNP-RESCUE-lm_741 Q11
 U 1 1 5CE90A8C
 P 7500 1950
@@
 $EndComp
 $Comp
-L eSim_NPN Q14
+L eSim_NPN-RESCUE-lm_741 Q14
 U 1 1 5CE90A8D
 P 7500 3050
@@
 $EndComp
 $Comp
-L eSim_NPN Q16
+L eSim_NPN-RESCUE-lm_741 Q16
 U 1 1 5CE90A91
 P 7050 3950
@@
 $EndComp
 $Comp
-L eSim_NPN Q15
+L eSim_NPN-RESCUE-lm_741 Q15
 U 1 1 5CE90A92
 P 7500 4300
@@
 $EndComp
 $Comp
-L eSim_NPN Q17
+L eSim_NPN-RESCUE-lm_741 Q17
 U 1 1 5CE90A95
 P 6800 4700
@@
 $EndComp
 $Comp
-L eSim_NPN Q18
+L eSim_NPN-RESCUE-lm_741 Q18
 U 1 1 5CE90A96
 P 8800 2300
@@
 $EndComp
 $Comp
-L eSim_NPN Q20
+L eSim_NPN-RESCUE-lm_741 Q20
 U 1 1 5CE90A97
 P 8400 2750
@@
 $EndComp
 $Comp
-L eSim_PNP Q19
+L eSim_PNP-RESCUE-lm_741 Q19
 U 1 1 5CE90A9A
 P 8800 4600

Commit message: Added gaw
Parts:
- Q1, Q12, Q13, Q14, Q15, Q16, Q17, Q18, Q2, Q20, Q3, Q7, Q8: symbol eSim_NPN-RESCUE-lm_741 -> eSim_NPN
- Q10, Q11, Q19, Q4, Q5, Q6, Q9: symbol eSim_PNP-RESCUE-lm_741 -> eSim_PNP
Changed lines of the file:
@@
 EESchema Schematic File Version 2
-LIBS:lm_741-rescue
 LIBS:power
 LIBS:eSim_Analog
@@
 LIBS:eSim_Plot
 LIBS:eSim_Power
-LIBS:eSim_User
+LIBS:eSim_PSpice
 LIBS:eSim_Sources
 LIBS:eSim_Subckt
+LIBS:eSim_User
 LIBS:lm_741-cache
 EELAYER 25 0
@@
 $EndDescr
 $Comp
-L eSim_NPN-RESCUE-lm_741 Q1
+L eSim_NPN Q1
 U 1 1 5CE90A7B
 P 2650 2700
@@
 $EndComp
 $Comp
-L eSim_NPN-RESCUE-lm_741 Q2
+L eSim_NPN Q2
 U 1 1 5CE90A7C
 P 4300 2700
@@
 $EndComp
 $Comp
-L eSim_PNP-RESCUE-lm_741 Q6
+L eSim_PNP Q6
 U 1 1 5CE90A7D
 P 3000 3200
@@
 $EndComp
 $Comp
-L eSim_PNP-RESCUE-lm_741 Q5
+L eSim_PNP Q5
 U 1 1 5CE90A7E
 P 3950 3200
@@
 $EndComp
 $Comp
-L eSim_NPN-RESCUE-lm_741 Q3
+L eSim_NPN Q3
 U 1 1 5CE90A7F
 P 3300 4000
@@
 $EndComp
 $Comp
-L eSim_PNP-RESCUE-lm_741 Q4
+L eSim_PNP Q4
 U 1 1 5CE90A80
 P 3850 2000
@@
 $EndComp
 $Comp
-L eSim_PNP-RESCUE-lm_741 Q9
+L eSim_PNP Q9
 U 1 1 5CE90A81
 P 5200 2000
@@
 $EndComp
 $Comp
-L eSim_NPN-RESCUE-lm_741 Q8
+L eSim_NPN Q8
 U 1 1 5CE90A82
 P 3950 4600
@@
 $EndComp
 $Comp
-L eSim_NPN-RESCUE-lm_741 Q7
+L eSim_NPN Q7
 U 1 1 5CE90A83
 P 3000 4600
@@
 $EndComp
 $Comp
-L eSim_NPN-RESCUE-lm_741 Q12
+L eSim_NPN Q12
 U 1 1 5CE90A87
 P 6300 4700
@@
 $EndComp
 $Comp
-L eSim_NPN-RESCUE-lm_741 Q13
+L eSim_NPN Q13
 U 1 1 5CE90A88
 P 5400 4700
@@
 $EndComp
 $Comp
-L eSim_PNP-RESCUE-lm_741 Q10
+L eSim_PNP Q10
 U 1 1 5CE90A8B
 P 6500 1950
@@
 $EndComp
 $Comp
-L eSim_PNP-RESCUE-lm_741 Q11
+L eSim_PNP Q11
 U 1 1 5CE90A8C
 P 7500 1950
@@
 $EndComp
 $Comp
-L eSim_NPN-RESCUE-lm_741 Q14
+L eSim_NPN Q14
 U 1 1 5CE90A8D
 P 7500 3050
@@
 $EndComp
 $Comp
-L eSim_NPN-RESCUE-lm_741 Q16
+L eSim_NPN Q16
 U 1 1 5CE90A91
 P 7050 3950
@@
 $EndComp
 $Comp
-L eSim_NPN-RESCUE-lm_741 Q15
+L eSim_NPN Q15
 U 1 1 5CE90A92
 P 7500 4300
@@
 $EndComp
 $Comp
-L eSim_NPN-RESCUE-lm_741 Q17
+L eSim_NPN Q17
 U 1 1 5CE90A95
 P 6800 4700
@@
 $EndComp
 $Comp
-L eSim_NPN-RESCUE-lm_741 Q18
+L eSim_NPN Q18
 U 1 1 5CE90A96
 P 8800 2300
@@
 $EndComp
 $Comp
-L eSim_NPN-RESCUE-lm_741 Q20
+L eSim_NPN Q20
 U 1 1 5CE90A97
 P 8400 2750
@@
 $EndComp
 $Comp
-L eSim_PNP-RESCUE-lm_741 Q19
+L eSim_PNP Q19
 U 1 1 5CE90A9A
 P 8800 4600
